File: hardware/jig/toorcamp2018jig.kicad_pcb (KiCad board)
At the start: 2 copper layers, 210 x 130 mm, 88 parts, among them J1 NEIGHBOR1, J2 NEIGHBOR2, J3 GOODFET, J4 TOP_INTERCONNECT, J5 BACK_INTERCONNECT, J6 FAULT, J7 BONUS_ROW, J8 TEST_2P, J9 TEST_2P, P1 CONN_01X02, P10 CONN_01X02, P11 CONN_01X02, P12 CONN_01X02, P13 CONN_01X02, P14 CONN_01X02, P2 CONN_01X02, P3 CONN_01X02, P4 CONN_01X02, P5 CONN_01X02, P6 CONN_01X02, P7 CONN_01X02, P8 CONN_01X02, P9 CONN_01X02, U1 NX5P2553GV

Commit message: filled in test jig bom info
Parts:
- U1: value NX5P2553GV -> AP2553W6-7
Connections:
- J1 pad 10: (no net) -> /P1_1
- J1 pad 11: (no net) -> /CLK0
- J1 pad 12: (no net) -> /P1_2
- J1 pad 3: (no net) -> /P4_9
- J1 pad 33: (no net) -> /P9_5
- J1 pad 34: (no net) -> /P9_6
- J1 pad 35: (no net) -> /P2_0
- J1 pad 36: (no net) -> /P6_0
- J1 pad 5: (no net) -> /P4_10
- J2 pad 11: (no net) -> /P4_7
- J2 pad 12: (no net) -> /CLK2
- J2 pad 13: (no net) -> /P2_8
- J2 pad 14: (no net) -> /P2_7
- J2 pad 15: (no net) -> /P2_6
- J2 pad 17: (no net) -> /WAKEUP0
- J2 pad 18: (no net) -> /P2_5
- J2 pad 19: (no net) -> /P2_4
- J2 pad 2: (no net) -> /VBUS
- J2 pad 20: (no net) -> /P2_3
- J2 pad 21: (no net) -> /PF_4
- J2 pad 22: (no net) -> /P3_2
- J2 pad 23: (no net) -> /P7_2
- J2 pad 24: (no net) -> /P3_1
- J2 pad 25: (no net) -> /P7_1
- J2 pad 26: (no net) -> /P3_0
- J2 pad 27: (no net) -> /P7_0
- J2 pad 29: (no net) -> /P6_8
- J2 pad 3: (no net) -> /P4_8
- J2 pad 30: (no net) -> /P3_7
- J2 pad 31: (no net) -> /P6_7
- J2 pad 32: (no net) -> /P3_3
- J2 pad 33: (no net) -> /P2_2
- J2 pad 34: (no net) -> /P6_6
- J2 pad 35: (no net) -> /P2_1
- J2 pad 36: (no net) -> /P6_3
- J2 pad 37: (no net) -> /P3_5
- J2 pad 38: (no net) -> /P3_6
- J2 pad 39: (no net) -> /I2C0_SDA
- J2 pad 40: (no net) -> /I2C0_SCL
- J3 pad 10: (no net) -> Net-(J3-Pad10)
- J3 pad 12: (no net) -> Net-(J3-Pad12)
- J3 pad 13: (no net) -> Net-(J3-Pad13)
- J3 pad 14: (no net) -> Net-(J3-Pad14)
- J3 pad 6: (no net) -> Net-(J3-Pad6)
- J7 pad 11: (no net) -> /RESET
- J7 pad 12: (no net) -> /VBAT
- J7 pad 13: (no net) -> /P2_11
- J7 pad 14: (no net) -> /P2_10
- J7 pad 15: (no net) -> /P6_10
- J7 pad 16: (no net) -> /P6_9
- J7 pad 17: (no net) -> /P6_2
- J7 pad 18: (no net) -> /P6_1
- J7 pad 2: (no net) -> /P6_4
- J7 pad 3: (no net) -> /P6_5
- J7 pad 4: (no net) -> /ADC0_5
- J7 pad 5: (no net) -> /ADC0_2
- J7 pad 6: (no net) -> /P2_9
- J7 pad 7: (no net) -> /P2_12
- J7 pad 8: (no net) -> /P2_13
- J7 pad 9: (no net) -> /RTC_ALARM
- P2 pad 1: (no net) -> Net-(P2-Pad1)
- P2 pad 2: (no net) -> Net-(P2-Pad2)
- P3 pad 1: (no net) -> Net-(P3-Pad1)
- P3 pad 2: (no net) -> Net-(P3-Pad2)
- P4 pad 1: (no net) -> Net-(P4-Pad1)
- P4 pad 2: (no net) -> Net-(P4-Pad2)
- P5 pad 1: (no net) -> Net-(P5-Pad1)
- P5 pad 2: (no net) -> Net-(P5-Pad2)
